Commit message: fix

File: src/pbot_description/urdf/pbot_ultrasound.xacro (robot description, xacro)
@@ -6,5 +6,5 @@
         <visual>
             <geometry>
-                <box size="0.01 0.01 0.02"/>
+                <box size="0.01 0.045 0.02 "/>
             </geometry>
             <material name="Red"/>
@@ -12,5 +12,5 @@
         <collision>
             <geometry>
-                <box size="0.01 0.045 0.02"/>
+                <box size="0.01 0.045 0.02 "/>
             </geometry>
         </collision>
@@ -24,5 +24,5 @@
         <parent link="base_link"/>
         <child link="pbot_ultrasonic"/>
-        <origin xyz="0.12 0 0.02" rpy="0 0 0"/> <!-- Позиция и ориентация датчика -->
+        <origin xyz="0.10 0 0.02" rpy="0 0 0"/> <!-- Позиция и ориентация датчика -->
     </joint>
     <!-- Определение датчика без плагина Gazebo -->
