Commit message: add lidar into gazebo

File: src/pbot_description/urdf/pbot_gazebo.xacro (robot description, xacro)
@@ -16,28 +16,31 @@
         <material>Gazebo/Green</material>
     </gazebo>
-<gazebo>
-    <plugin name="gazebo_ros_joint_state_publisher" filename="libgazebo_ros_joint_state_publisher.so">
-        <update_rate>20</update_rate>
-        <jointName>pbot_rf_w_to_base, pbot_rr_w_to_base, pbot_lf_w_to_base, pbot_lr_w_to_base</jointName>
-<!--        <jointName>pbot_rr_w_to_base</jointName>-->
-<!--        <jointName>pbot_lf_w_to_base</jointName>-->
-<!--        <jointName>pbot_lr_w_to_base</jointName>-->
-    </plugin>
-</gazebo>
-<!--    -->
-<!--  <gazebo>-->
-<!--    <plugin name="gazebo_ros_control" filename="libgazebo_ros_control.so">-->
-<!--      <robotNamespace>/</robotNamespace>-->
-<!--    </plugin>-->
-<!--  </gazebo>-->
-<!--    <gazebo>-->
-<!--        <plugin name="gazebo_ros_joint_state_publisher"-->
-<!--            filename="libgazebo_ros_joint_state_publisher.so">-->
-<!--            <update_rate>20</update_rate>-->
-<!--            <joint_name>pbot_lf_w_to_base</joint_name>-->
-<!--            <joint_name>pbot_lr_w_to_base</joint_name>-->
-<!--            <joint_name>pbot_rf_w_to_base</joint_name>-->
-<!--            <joint_name>pbot_rr_w_to_base</joint_name>-->
-<!--        </plugin>-->
-<!--    </gazebo>-->
+    <gazebo reference="laser_frame">
+        <material>Gazebo/Red</material>
+    </gazebo>
+    <gazebo>
+        <plugin name="gazebo_ros_joint_state_publisher" filename="libgazebo_ros_joint_state_publisher.so">
+            <update_rate>20</update_rate>
+            <jointName>pbot_rf_w_to_base, pbot_rr_w_to_base, pbot_lf_w_to_base, pbot_lr_w_to_base</jointName>
+            <!--        <jointName>pbot_rr_w_to_base</jointName>-->
+            <!--        <jointName>pbot_lf_w_to_base</jointName>-->
+            <!--        <jointName>pbot_lr_w_to_base</jointName>-->
+        </plugin>
+    </gazebo>
+    <!--    -->
+    <!--  <gazebo>-->
+    <!--    <plugin name="gazebo_ros_control" filename="libgazebo_ros_control.so">-->
+    <!--      <robotNamespace>/</robotNamespace>-->
+    <!--    </plugin>-->
+    <!--  </gazebo>-->
+    <!--    <gazebo>-->
+    <!--        <plugin name="gazebo_ros_joint_state_publisher"-->
+    <!--            filename="libgazebo_ros_joint_state_publisher.so">-->
+    <!--            <update_rate>20</update_rate>-->
+    <!--            <joint_name>pbot_lf_w_to_base</joint_name>-->
+    <!--            <joint_name>pbot_lr_w_to_base</joint_name>-->
+    <!--            <joint_name>pbot_rf_w_to_base</joint_name>-->
+    <!--            <joint_name>pbot_rr_w_to_base</joint_name>-->
+    <!--        </plugin>-->
+    <!--    </gazebo>-->
 </robot>
