Commit message: fix

File: src/pbot_description/urdf/pbot.xacro (robot description, xacro)
@@ -6,4 +6,13 @@
     <xacro:include filename="$(find pbot_description)/urdf/pbot_materials.xacro"/>
     <xacro:property name="clearance" value="0.043" />
+    <!-- base_link -->
+    <link name="base_link">
+        <visual>
+            <origin xyz="0 0 0" rpy="0 0 0"/>
+            <geometry>
+                <sphere radius="0.001"/>
+            </geometry>
+        </visual>
+    </link>
     <!-- base_footprint -->
     <link name="base_footprint">
@@ -16,18 +25,9 @@
         </visual>
     </link>
-    <joint name="base_footprint_to_base_link" type="fixed">
-        <origin xyz="0 0 ${clearance}" rpy="0 0 0" />
-        <parent link="base_footprint" />
-        <child link="base_link" />
+    <joint name="base_link_to_base_footprint" type="fixed">
+        <origin xyz="0 0 -${clearance}" rpy="0 0 0" />
+        <parent link="base_link" />
+        <child link="base_footprint" />
     </joint>
-    <!-- base_link -->
-    <link name="base_link">
-        <visual>
-            <origin xyz="0 0 0" rpy="0 0 0"/>
-            <geometry>
-                <sphere radius="0.001"/>
-            </geometry>
-        </visual>
-    </link>
     <joint name="base_link_to_pbot_base" type="fixed">
         <origin xyz="0 0 0" rpy="0 0 0"/>

Commit message: add range bound

File: src/pbot_description/urdf/pbot.xacro (robot description, xacro)
@@ -5,5 +5,5 @@
     <!-- Matherials -->
     <xacro:include filename="$(find pbot_description)/urdf/pbot_materials.xacro"/>
-    <xacro:property name="clearance" value="0.043" />
+    <xacro:property name="clearance" value="0.043"/>
     <!-- base_link -->
     <link name="base_link">
@@ -14,19 +14,33 @@
             </geometry>
         </visual>
+        <inertial>
+            <origin
+                    xyz="-0.0126793836830341 4.44350410814448E-10 -0.00681296059112218"
+                    rpy="0 0 0"/>
+            <mass
+                    value="0.28831638977324"/>
+            <inertia
+                    ixx="0.000131169085410887"
+                    ixy="-4.3600054751417E-15"
+                    ixz="9.31897878301522E-06"
+                    iyy="0.000567748496773017"
+                    iyz="-9.53741865535676E-15"
+                    izz="0.000682526229970573"/>
+        </inertial>
     </link>
     <!-- base_footprint -->
     <link name="base_footprint">
         <visual>
-            <origin xyz="0 0 0" rpy="0 0 0" />
+            <origin xyz="0 0 0" rpy="0 0 0"/>
             <geometry>
-                <cylinder length="0.001" radius="0.110" />
+                <cylinder length="0.001" radius="0.110"/>
             </geometry>
-            <material name="Blue" />
+            <material name="Blue"/>
         </visual>
     </link>
     <joint name="base_link_to_base_footprint" type="fixed">
-        <origin xyz="0 0 -${clearance}" rpy="0 0 0" />
-        <parent link="base_link" />
-        <child link="base_footprint" />
+        <origin xyz="0 0 -${clearance}" rpy="0 0 0"/>
+        <parent link="base_link"/>
+        <child link="base_footprint"/>
     </joint>
     <joint name="base_link_to_pbot_base" type="fixed">
@@ -76,9 +90,11 @@
     </link>
     <!-- Ultrasound -->
-    <xacro:include filename="$(find pbot_description)/urdf/pbot_ultrasound.xacro" />
+    <xacro:include filename="$(find pbot_description)/urdf/pbot_ultrasound.xacro"/>
     <!-- Wheels -->
-    <xacro:include filename="$(find pbot_description)/urdf/pbot_rf_w.xacro" />
-    <xacro:include filename="$(find pbot_description)/urdf/pbot_rr_w.xacro" />
-    <xacro:include filename="$(find pbot_description)/urdf/pbot_lf_w.xacro" />
-    <xacro:include filename="$(find pbot_description)/urdf/pbot_lr_w.xacro" />
+    <xacro:include filename="$(find pbot_description)/urdf/pbot_rf_w.xacro"/>
+    <xacro:include filename="$(find pbot_description)/urdf/pbot_rr_w.xacro"/>
+    <xacro:include filename="$(find pbot_description)/urdf/pbot_lf_w.xacro"/>
+    <xacro:include filename="$(find pbot_description)/urdf/pbot_lr_w.xacro"/>
+    <!-- Gazebo -->
+    <xacro:include filename="$(find pbot_description)/urdf/pbot_gazebo.xacro"/>
 </robot>

Commit message: change model

File: src/pbot_description/urdf/pbot.xacro (robot description, xacro)
@@ -53,15 +53,15 @@
         <inertial>
             <origin
-                    xyz="-0.0126793836830341 4.44350410814448E-10 -0.00681296059112218"
+                    xyz="-0.00021219 -0.001448 0.037164"
                     rpy="0 0 0"/>
             <mass
-                    value="0.28831638977324"/>
+                    value="0.88805"/>
             <inertia
-                    ixx="0.000131169085410887"
-                    ixy="-4.3600054751417E-15"
-                    ixz="9.31897878301522E-06"
-                    iyy="0.000567748496773017"
-                    iyz="-9.53741865535676E-15"
-                    izz="0.000682526229970573"/>
+                    ixx="0.00053126"
+                    ixy="-3.6522E-07"
+                    ixz="1.6178E-05"
+                    iyy="0.0011501"
+                    iyz="-1.8024E-08"
+                    izz="0.0016371"/>
         </inertial>
         <visual>
@@ -75,6 +75,6 @@
             <material
                     name="White">
-                <!--                <color-->
-                <!--                        rgba="0.698039215686274 0.698039215686274 0.698039215686274 1"/>-->
+<!--                <color-->
+<!--                        rgba="0.69804 0.69804 0.69804 1"/>-->
             </material>
         </visual>
@@ -92,5 +92,7 @@
     <xacro:include filename="$(find pbot_description)/urdf/pbot_lidar.xacro"/>
     <!-- Ultrasound -->
-    <xacro:include filename="$(find pbot_description)/urdf/pbot_ultrasound.xacro"/>
+    <xacro:include filename="$(find pbot_description)/urdf/pbot_sonar.xacro"/>
+    <!-- Camera -->
+    <xacro:include filename="$(find pbot_description)/urdf/pbot_camera.xacro"/>
     <!-- Wheels -->
     <xacro:include filename="$(find pbot_description)/urdf/pbot_rf_w.xacro"/>

File: src/pbot_description/urdf/pbot_lf_w.xacro (robot description, xacro)
@@ -7,15 +7,15 @@
         <inertial>
             <origin
-                    xyz="2.2904E-10 -0.00027973 -1.3045E-10"
+                    xyz="2.20207470313927E-10 -0.000279731201700426 -2.0205375914073E-10"
                     rpy="0 0 0"/>
             <mass
-                    value="0.030238"/>
+                    value="0.0302375576064607"/>
             <inertia
-                    ixx="1.157E-05"
-                    ixy="6.3103E-14"
-                    ixz="-1.9026E-14"
-                    iyy="1.9609E-05"
-                    iyz="-5.1829E-14"
-                    izz="1.157E-05"/>
+                    ixx="1.15702197035643E-05"
+                    ixy="5.87881486177672E-14"
+                    ixz="1.10485738589503E-14"
+                    iyy="1.96090957656786E-05"
+                    iyz="-6.70315528384273E-14"
+                    izz="1.15702193827656E-05"/>
         </inertial>
         <visual>
@@ -43,6 +43,6 @@
             type="continuous">
         <origin
-                xyz="0.045046 0.0705 -0.013263"
-                rpy="0 0.016895 0"/>
+                xyz="0.0470881159981717 0.0705 -0.0132839044168557"
+                rpy="0 0.0166094578206922 0"/>
         <parent
                 link="pbot_base"/>

File: src/pbot_description/urdf/pbot_lidar.xacro (robot description, xacro)
@@ -3,24 +3,52 @@
         xmlns:xacro="http://www.ros.org/wiki/xacro"
         name="pbot">
-    <joint name="laser_joint" type="fixed">
-        <parent link="base_link"/>
-        <child link="laser_frame"/>
-        <origin xyz="0 0 0.05" rpy="0 0 0"/>
-    </joint>
-    <link name="laser_frame">
+    <link
+            name="laser_frame">
+        <inertial>
+            <origin
+                    xyz="0.00208191942450915 3.97647389113363E-18 -0.00385299208880718"
+                    rpy="0 0 0"/>
+            <mass
+                    value="0.968613348864223"/>
+            <inertia
+                    ixx="0.000334583006933795"
+                    ixy="-5.24034614619688E-20"
+                    ixz="1.81259849319653E-21"
+                    iyy="0.000411095059912044"
+                    iyz="-3.29708352475897E-21"
+                    izz="0.000675110546906932"/>
+        </inertial>
         <visual>
+            <origin
+                    xyz="0 0 0"
+                    rpy="0 0 0"/>
             <geometry>
-                <cylinder radius="0.015" length="0.01"/>
+                <mesh
+                        filename="package://pbot_description/meshes/laser_frame.STL"/>
             </geometry>
             <material name="Red"/>
         </visual>
         <collision>
+            <origin
+                    xyz="0 0 0"
+                    rpy="0 0 0"/>
             <geometry>
-                <cylinder radius="0.015" length="0.01"/>
+                <mesh
+                        filename="package://pbot_description/meshes/laser_frame.STL"/>
             </geometry>
         </collision>
-        <!--    <xacro:inertial_cylinder mass="0.1" length="0.04" radius="0.05">-->
-        <!--        <origin xyz="0 0 0" rpy="0 0 0"/>-->
-        <!--    </xacro:inertial_cylinder>-->
     </link>
+    <joint
+            name="laser_joint"
+            type="fixed">
+        <origin
+                xyz="0.0039648 0 0.12415"
+                rpy="0 -0.016609 3.1416"/>
+        <parent
+                link="pbot_base"/>
+        <child
+                link="laser_frame"/>
+        <axis
+                xyz="0 0 0"/>
+    </joint>
 </robot>

File: src/pbot_description/urdf/pbot_lr_w.xacro (robot description, xacro)
@@ -7,15 +7,15 @@
         <inertial>
             <origin
-                    xyz="-1.3858E-10 -0.00027973 1.3827E-10"
+                    xyz="3.29489630024327E-11 -0.0002797313481048 -1.85563862886706E-10"
                     rpy="0 0 0"/>
             <mass
-                    value="0.030238"/>
+                    value="0.0302375580133055"/>
             <inertia
-                    ixx="1.157E-05"
-                    ixy="-3.977E-14"
-                    ixz="5.9664E-14"
-                    iyy="1.9609E-05"
-                    iyz="1.6868E-14"
-                    izz="1.157E-05"/>
+                    ixx="1.15702196840428E-05"
+                    ixy="-2.03000444280046E-14"
+                    ixz="1.06746865771734E-13"
+                    iyy="1.96090960377303E-05"
+                    iyz="-5.58321097468027E-14"
+                    izz="1.15702197584359E-05"/>
         </inertial>
         <visual>
@@ -43,6 +43,6 @@
             type="continuous">
         <origin
-                xyz="-0.074937 0.0705 -0.011236"
-                rpy="0 0.016895 0"/>
+                xyz="-0.0728953319370116 0.0705 -0.0112908611194895"
+                rpy="0 0.0166094578206921 0"/>
         <parent
                 link="pbot_base"/>

File: src/pbot_description/urdf/pbot_rf_w.xacro (robot description, xacro)
@@ -7,5 +7,5 @@
         <inertial>
             <origin
-                    xyz="2.9058E-11 0.00027973 5.9298E-10"
+                    xyz="7.0441E-11 0.00027973 4.457E-10"
                     rpy="0 0 0"/>
             <mass
@@ -13,8 +13,8 @@
             <inertia
                     ixx="1.157E-05"
-                    ixy="7.6572E-15"
-                    ixz="-8.7242E-14"
+                    ixy="-7.5717E-15"
+                    ixz="-3.0141E-14"
                     iyy="1.9609E-05"
-                    iyz="-1.3863E-13"
+                    iyz="-1.0612E-13"
                     izz="1.157E-05"/>
         </inertial>
@@ -43,6 +43,6 @@
             type="continuous">
         <origin
-                xyz="0.045046 -0.0705 -0.013263"
-                rpy="0 0.016895 0"/>
+                xyz="0.047088 -0.0705 -0.013284"
+                rpy="0 0.016609 0"/>
         <parent
                 link="pbot_base"/>

File: src/pbot_description/urdf/pbot_rr_w.xacro (robot description, xacro)
@@ -7,15 +7,15 @@
         <inertial>
             <origin
-                    xyz="5.388E-10 0.00027973 5.4071E-10"
+                    xyz="5.38798672344853E-10 0.00027973133311894 5.4071500402153E-10"
                     rpy="0 0 0"/>
             <mass
-                    value="0.030238"/>
+                    value="0.0302375580628956"/>
             <inertia
-                    ixx="1.157E-05"
-                    ixy="-1.3445E-13"
-                    ixz="-3.6496E-14"
-                    iyy="1.9609E-05"
-                    iyz="-1.236E-13"
-                    izz="1.157E-05"/>
+                    ixx="1.15702196703268E-05"
+                    ixy="-1.34449266129171E-13"
+                    ixz="-3.64897808319972E-14"
+                    iyy="1.96090960765893E-05"
+                    iyz="-1.23593693591465E-13"
+                    izz="1.1570219796082E-05"/>
         </inertial>
         <visual>
@@ -43,6 +43,6 @@
             type="continuous">
         <origin
-                xyz="-0.074937 -0.0705 -0.011236"
-                rpy="0 0.016895 0"/>
+                xyz="-0.0728953319370115 -0.0705 -0.0112908611194895"
+                rpy="0 0.0166094578206924 0"/>
         <parent
                 link="pbot_base"/>
